File: atkeyboard/atkeyboard.kicad_pcb (KiCad board)
At the start: 2 copper layers, 112 x 62 mm, 76 parts, among them J1 AT328P-ProgPins, J2 ComClav, J3 SW_Push_45deg, K1 SW_Push_45deg, M1 SW_Push_45deg, P1 SW_Push_45deg, Q1 SW_Push_45deg, T1 SW_Push_45deg, U1 ATmega328P-AU, U2 SW_Push_45deg, X1 SW_Push_45deg, Y2 SW_Push_45deg

Commit message: Add files via upload
Parts:
- added IC1: ADXL345, 18650:ADXL345, F.Cu at (143.9, 95.7)
- added J4: INTx, 18650:2PADS, B.Cu at (129.6, 94.2)
- added R3: PUPSDA, Resistors_SMD:R_0805_HandSoldering, F.Cu at (160.8, 98.0)
- added R4: PUPSDA, Resistors_SMD:R_0805_HandSoldering, F.Cu at (155.8, 98.0)
- Y1: renamed from 8 Mhz
- moved G*** 0.84 mm to (185.8, 138.7)
- moved G*** 0.77 mm to (185.6, 138.5)
Routing:
- net Net-(IC1-Pad9): track 0.00 -> 92.1 mm, vias 0 -> 7
- net +3V3: track 160.3 -> 233.1 mm, vias 1 -> 11
- net /SCL: track 28.1 -> 97.3 mm, vias 1 -> 6
- net /SDA: track 37.5 -> 67.7 mm, vias 1 -> 2
- net Net-(IC1-Pad8): track 0.00 -> 18.5 mm, vias 0 -> 1
- net /C3: track 210.9 -> 221.7 mm, vias 3 -> 10
- net GND: track 317.7 -> 325.6 mm, vias 35 -> 37
- net /C1: track 158.6 -> 163.4 mm
- net /R5: track 277.8 -> 282.3 mm
- net (no net): vias 45 -> 44
Other:
- board text added: "ADXL345"
- board text added: "Dr CADIC Philippe"
- board text added: "I2C Pullups"
- board text added: "Small I2C Keyboard Based on ATMega328P-AU"
- board text added: "V1.0"
- board text added: "https://github.com/ccadic/atmega328kb"
